File: MDB1986.brd (EAGLE design)
At the start: 100 x 80 mm, 113 parts, among them IC1 MAX3232CSE, J1 USB-TYPE-B, J2 USB-TYPE-B, U2 IS61LV25616AL, U3 STM32F103CBT6-LQFP48, U4 MAX7221CWG, U5 AMS1117-3.3, U6 MCP2551, X1 DRB-9FA, X2 DRB-9MA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

Commit message: Add files via upload
Parts:
- U7: value (none) -> W25Q64FV
- moved C2 4.61 mm to (68.5, 14.0), turned to 270 degrees
- moved R4 2.00 mm to (18.0, 52.0)
- moved R5 2.00 mm to (18.0, 50.0)
- moved R23 1.00 mm to (71.0, 14.0), turned to 270 degrees
- renumbered IC1 to U8
Connections:
- net N$26: now also R3.2
- net STUSB_DM: no longer R3.2
Routing:
- net GND: track 682.0 -> 686.7 mm, vias 34 -> 35
- net STUSB_DM: track 5.61 -> 8.72 mm
- net N$25: track 17.5 -> 15.3 mm
- net STUSB_DP: track 8.51 -> 6.79 mm
- net CAN_H: track 23.5 -> 25.1 mm
- net N$26: track 20.1 -> 21.4 mm
- net N$42: track 11.9 -> 10.7 mm
- net N$45: track 22.6 -> 23.3 mm
Other:
- board text added: "PB0 D16 IN1+ T3.C1 Btn1 PB1 D17 IN1- T3.C1N Btn2 PB2 D18 IN2+ T3.C2 Led PB3 D19 IN2- T3.C2N Led PB4 D20 IN3+ T3.C3 Led PB5 D21 IN3- T3.C3N Led PB6 D22 IN4+ T3.C4 Led PC3 U1.TX CLE IR1.Out PC4 U1.RX BSY IR1.In"
- board text added: "PB11 D27 IN6- T2.C2N w25CS PD1 PRDA+ CLE A15 RAM PD2 PRDA- S1.TX A14 RAM PC9 S2.TX BE0 Can1.RX PC10 S2.RX BE1 Can1.TX PC11 S2.CK BE2 Can2.RX PC12 S2.FS BE3 Can2.TX PC13 PRMA+ A30 U2.TX PC14 PRMA- A31 U2.RX"
- board text added: "PD10 S2.FSS RTS2 A1 UART2 PD11 A0 CTS2 UART2 PD13 U2.TX Out1+ IR2.Out UART2 PD14 U2.RX Out1- IR2.In UART2 PE2 Out4- A16 DAC1 PE11 Can1.RX A25 CAN1 PE12 Can1.TX A26 CAN1 PE13 Can2.RX A27 PE14 Can2.TX A28"
- board text added: "PD9 S2.SCK DSR2 A2 ADC2 PC5 Ext1 S1.TX S1.RX SSP1 PC6 Ext2 S1.RX S1.TX SSP1 PC7 Ext3 S1.CK FXEN SSP1 PC8 Ext4 S1.FS FTX PF3 PRMC+ A0 T1.CH1 PF4 PRMC- A1 T1.CH2 RAM PF7 PRDC+ A4 Out4+ RAM PF8 PRDC- A5 Out4- RAM"
- board text removed: "D:/1/Il-96M.bmp"
- board text removed: "PB0 D16 IN1+ T3.C1 Btn1 PB1 D17 IN1- T3.C1N Btn2 PB2 D18 IN2+ T3.C2 Led PB3 D19 IN2- T3.C2N Led PB4 D20 IN3+ T3.C3 Led PB5 D21 IN3- T3.C3N Led PB6 D22 IN4+ T3.C4 Led PC3 UTX1 CLE IR1.O PC4 URX1 BSY IR1.In"
- board text removed: "PB11 D27 IN6- T2.C2N w25CS PD1 PRDA+ CLE A15 RAM PD2 PRDA- S1.TX A14 RAM PC9 S2.TX BE0 CanRX1 PC10 S2.RX BE1 CanTX1 PC11 S2.CK BE2 CanRX2 PC12 S2.FS BE3 CanTX2 PC13 PRMA+ A30 UTX2 PC14 PRMA- A31 URX2"
- board text removed: "PD10 S2.FSS RTS2 A1 rs232 PD11 A0 CTS2 rs232 PD13 UTX2 Out1+ IR2.O rs232 PD14 URX2 Out1- IR2.In rs232 PE2 Out4- A16 DAC1 PE11 Can.RX1 A25 CAN PE12 Can.TX1 A26 CAN PE13 Can.RX2 A27 PE14 Can.TX2 A28"
- board text removed: "PD9 S2.SCK DSR2 A2 ADC2 PC5 Ext1 S1.TX S1.RX MOSI PC6 Ext2 S1.RX S1.TX MISO PC7 Ext3 S1.CK FXEN CLK PC8 Ext4 S1.FS FTX PF3 PRMC+ A0 T1.CH1 PF4 PRMC- A1 T1.CH2 RAM PF7 PRDC+ A4 Out4+ RAM PF8 PRDC- A5 Out4- RAM"
- board text removed: "ver. 1.0"
