File: MDB1986.sch (EAGLE design)
At the start: 113 parts, among them IC1 MAX3232CSE, J1 USB-TYPE-B, J2 USB-TYPE-B, U2 IS61LV25616AL, U3 STM32F103CBT6-LQFP48, U4 MAX7221CWG, U5 AMS1117-3.3, U6 MCP2551, X1 DRB-9FA, X2 DRB-9MA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

Commit message: Add files via upload
Parts:
- U7: value (none) -> W25Q64FV
- renumbered IC1 to U8
Connections:
- net N$26: now also R3.2
- net STUSB_DM: no longer R3.2
Other:
- moved on the sheet: D3, F2, R3, R4, R5
